File: pcb/hdmi-breakout/hdmi-breakout.kicad_pcb (KiCad board)
At the start: 4 copper layers, 35 x 29 mm, 6 parts, among them J1 Conn_01x09, J2 HDMI_A_1.4, J3 HDMI_A_1.4, J4 Conn_01x09

Commit message: update hardware
Other:
- board text added: "github.com/flaviut/ceclink"
- board text removed: "github.com/gkoh/pico-cec"
